File: pcb/pcb.kicad_pcb (KiCad board)
At the start: 2 copper layers, 4 parts, among them SW1 KEY_SW

Commit message: update: last updated
Parts:
- removed BT1: CR1216, Battery:BatteryHolder_LINX_BAT-HLD-012-SMT
- added B1: LR44, Battery:BatteryHolder_Keystone_2998_1x6.8mm, B.Cu at (21.1, 20.9)
- added G***: LOGO, LOGO, F.Cu at (15.4, 14.8)
- D1: footprint LED_SMD:LED_0603_1608Metric -> LED_SMD:LED_0402_1005Metric
- R1: footprint Resistor_SMD:R_0201_0603Metric -> LED_SMD:LED_0201_0603Metric
- moved R1 164.9 mm to (18.0, 22.6)
- moved D1 164.4 mm to (21.1, 25.1)
- moved SW1 164.2 mm to (23.7, 15.9)
Connections:
- D1 pad 1: GND -> Net-(D1-K)
- SW1 pad 1: +3.0V -> Net-(B1-Pad+)
Routing:
- net Net-(R1-Pad2): track 5.26 -> 4.08 mm
- net Net-(D1-A): track 3.09 -> 4.21 mm
- net Net-(D1-K): vias 0 -> 1
- net (no net): vias 1 -> 0
Other:
- board outline added: 12.5 x 12.5 mm
- board text added: "덕영고등학교 소프트웨어부."

Commit message: update: pcb update
Parts:
- removed B1: LR44, Battery:BatteryHolder_Keystone_2998_1x6.8mm
- added ?: , , F.Cu at (21.1, 15.7)
- added REF**: Banana_Jack_1Pin, Connector:Banana_Jack_1Pin, F.Cu at (21.1, 25.5)
- R1: value ~ -> 47
- moved D1 1.15 mm to (21.1, 23.9)
- moved R1 0.75 mm to (18.0, 21.8)
- moved G*** 0.05 mm to (15.3, 14.8)
Routing:
- net Net-(D1-A): track 4.21 -> 3.35 mm
- net Net-(R1-Pad2): track 4.08 -> 3.33 mm

Commit message: update: pcb update
Parts:
- moved G*** 13.7 mm to (22.5, 26.5)

Commit message: update: pcb update
Parts:
- moved G*** 0.45 mm to (22.6, 26.1)
Other:
- outline, holes or cut-outs redrawn

Commit message: update: update
Parts:
- D1: value LED -> BLUE
Other:
- board text added: "덕영고등학교 MAKE동아리"
- board text removed: "덕영고등학교 소프트웨어부."

Commit message: update: update
Parts:
- G***: moved to B.Cu
- R1: footprint LED_SMD:LED_0201_0603Metric -> Resistor_SMD:R_0603_1608Metric
- moved REF** 2.71 mm to (19.0, 23.8)
- moved ? 2.71 mm to (19.0, 14.0)
- moved SW1 2.71 mm to (21.5, 14.2)
- moved D1 2.71 mm to (19.0, 22.2)
- moved G*** 2.69 mm to (23.7, 23.6), turned to 180 degrees
- moved R1 2.06 mm to (17.2, 23.7), turned to -90 degrees
Routing:
- net Net-(R1-Pad2): track 3.33 -> 9.00 mm
- net Net-(D1-K): track 0.00 -> 1.54 mm
- net Net-(D1-A): track 3.35 -> 1.85 mm
Other:
- board text added: "B"
- board text added: "DYHS MAKE"
- board text added: "F"
- board text removed: "덕영고등학교 MAKE동아리"
