File: pcb/pcb.kicad_sch (KiCad schematic)
At the start: 4 parts, among them SW1 KEY_SW

Commit message: update: last updated
Parts:
- removed BT1: CR1216, Battery:BatteryHolder_LINX_BAT-HLD-012-SMT, symbol Device:Battery_Cell
- added B1: LR44, Battery:BatteryHolder_Keystone_2998_1x6.8mm, symbol LR44:LR44
- D1: footprint LED_SMD:LED_0603_1608Metric -> LED_SMD:LED_0402_1005Metric
- R1: value ~ -> 47; footprint Resistor_SMD:R_0201_0603Metric -> LED_SMD:LED_0201_0603Metric
Connections:
- net +3.0V: no longer names the net of SW1.1
- net +3.0V: now also B1.+
- net GND: no longer names the net of D1.1 (K)
- net GND: now also B1.-

Commit message: update: pcb update
Parts:
- B1: value LR44 -> 3V; footprint Battery:BatteryHolder_Keystone_2998_1x6.8mm -> Battery:BatteryHolder_LINX_BAT-HLD-012-SMT
Changed lines of the file:
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@@
 			)
 		)
-		(property "Value" "LR44"
+		(property "Value" "3V"
 			(at 165.1 95.2499 90)
 			(effects
@@
 			)
 		)
-		(property "Footprint" "Battery:BatteryHolder_Keystone_2998_1x6.8mm"
+		(property "Footprint" "Battery:BatteryHolder_LINX_BAT-HLD-012-SMT"
 			(at 161.29 93.98 0)
 			(effects

Commit message: update: update
Parts:
- D1: value LED -> BLUE
Changed lines of the file:
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@@
 (kicad_sch
-	(version 20231120)
+	(version 20250114)
 	(generator "eeschema")
-	(generator_version "8.0")
+	(generator_version "9.0")
 	(paper "A4")
 	(title_block
@@
 			)
 		)
-		(property "Value" "LED"
+		(property "Value" "BLUE"
 			(at 139.7 108.2674 90)
 			(effects
@@
 		)
 	)
+	(embedded_fonts no)
 )

Commit message: update: update
Parts:
- R1: footprint LED_SMD:LED_0201_0603Metric -> Resistor_SMD:R_0603_1608Metric
Changed lines of the file:
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@@
 			)
 		)
-		(property "Footprint" "LED_SMD:LED_0201_0603Metric"
+		(property "Footprint" "Resistor_SMD:R_0603_1608Metric"
 			(at 137.668 93.98 90)
 			(effects
